File: MDR32-K1986BE92FI-DK/MDR32-K1986BE92FI-DK.kicad_sch (KiCad schematic)
At the start: 57 parts, among them J1 Conn_PROBE, J2 PIN_A, J3 SYS_A, J4 USB_C_Receptacle_USB2.0_16P, J5 PIN_B, J6 SYS_B, Q1 AO3401A, SW1 IT-1181, SW2 SW_DIP_x02, SW3 IT-1181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

Commit message: fix probe connector
Parts:
- removed J1: Conn_PROBE, Connector_PinHeader_2.54mm:PinHeader_1x05_P2.54mm_Vertical, symbol Connector_Generic:Conn_01x05
- added J7: Conn_PROBE, symbol Connector_Generic:Conn_01x04
Connections:
- net +3V3_SRC: now also J7.1 (Pin_1)
- net GND: now also J7.4 (Pin_4)
- net JATCK: now also J7.3 (Pin_3)
- net JATMS: now also J7.2 (Pin_2)

Commit message: symbol rename and fixed
Parts:
- J1: renamed from J7; footprint (none) -> Connector_PinHeader_2.54mm:PinHeader_1x04_P2.54mm_Vertical
- renumbered D6 to D5
Changed lines of the file:
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@@
 		(on_board yes)
 		(dnp no)
-		(property "Reference" "D6"
+		(property "Reference" "D5"
 			(at 200.9774 102.87 0)
 			(effects
@@
 			(project "MDR32-K1986BE92FI-DK"
 				(path "/5712a142-8ffb-41af-8f2a-b31937ef9df4"
-					(reference "D6")
+					(reference "D5")
 					(unit 1)
 				)
@@
 		(on_board yes)
 		(dnp no)
-		(fields_autoplaced yes)
-		(property "Reference" "J7"
+		(property "Reference" "J1"
 			(at 199.39 34.2899 0)
 			(effects
@@
 			)
 		)
-		(property "Footprint" ""
+		(property "Footprint" "Connector_PinHeader_2.54mm:PinHeader_1x04_P2.54mm_Vertical"
 			(at 196.85 34.29 0)
 			(effects
@@
 			(project ""
 				(path "/5712a142-8ffb-41af-8f2a-b31937ef9df4"
-					(reference "J7")
+					(reference "J1")
 					(unit 1)
 				)
@@
 		(dnp no)
 		(fields_autoplaced yes)
-		(property "Reference" "#PWR032"
+		(property "Reference" "#PWR031"
 			(at 186.69 176.53 0)
 			(effects
@@
 			(project "MDR32-K1986BE92FI-DK"
 				(path "/5712a142-8ffb-41af-8f2a-b31937ef9df4"
-					(reference "#PWR032")
+					(reference "#PWR031")
 					(unit 1)
 				)
@@
 		(dnp no)
 		(fields_autoplaced yes)
-		(property "Reference" "#PWR054"
+		(property "Reference" "#PWR032"
 			(at 189.23 33.02 0)
 			(effects
@@
 			(project "MDR32-K1986BE92FI-DK"
 				(path "/5712a142-8ffb-41af-8f2a-b31937ef9df4"
-					(reference "#PWR054")
+					(reference "#PWR032")
 					(unit 1)
 				)
@@
 		(dnp no)
 		(fields_autoplaced yes)
-		(property "Reference" "#PWR033"
+		(property "Reference" "#PWR034"
 			(at 189.23 72.39 0)
 			(effects
@@
 			(project "MDR32-K1986BE92FI-DK"
 				(path "/5712a142-8ffb-41af-8f2a-b31937ef9df4"
-					(reference "#PWR033")
+					(reference "#PWR034")
 					(unit 1)
 				)
@@
 		(dnp no)
 		(fields_autoplaced yes)
-		(property "Reference" "#PWR055"
+		(property "Reference" "#PWR033"
 			(at 189.23 48.26 0)
 			(effects
@@
 			(project "MDR32-K1986BE92FI-DK"
 				(path "/5712a142-8ffb-41af-8f2a-b31937ef9df4"
-					(reference "#PWR055")
+					(reference "#PWR033")
 					(unit 1)
 				)

Commit message: change pinout on header
Connections:
- net +3V3_SRC: now also J3.2 (Pin_2); no longer J3.8 (Pin_8)
- net +BATT_SRC: now also J3.3 (Pin_3); no longer J3.7 (Pin_7)
- net GND: now also J2.1 (Pin_1), J2.2 (Pin_2), J3.1 (Pin_1), J6.1 (Pin_1); no longer J2.15 (Pin_15), J2.16 (Pin_16), J3.10 (Pin_10), J6.10 (Pin_10)
- net JATCK: now also J3.8 (Pin_8); no longer J3.3 (Pin_3)
- net JATDI: now also J3.7 (Pin_7); no longer J3.4 (Pin_4)
- net JATDO: now also J3.10 (Pin_10); no longer J3.1 (Pin_1)
- net JATMS: now also J3.9 (Pin_9); no longer J3.2 (Pin_2)
- net JAnTRS: now also J3.6 (Pin_6); no longer J3.5 (Pin_5)
- net JBTCK: now also J6.8 (Pin_8); no longer J6.4 (Pin_4)
- net JBTDI: now also J6.7 (Pin_7); no longer J6.5 (Pin_5)
- net JBTDO: now also J6.10 (Pin_10); no longer J6.2 (Pin_2)
- net JBTMS: now also J6.9 (Pin_9); no longer J6.3 (Pin_3)
- net PA0: now also J2.16 (Pin_16); no longer J2.1 (Pin_1)
- net PA1: now also J2.15 (Pin_15); no longer J2.2 (Pin_2)
- net PA2: now also J2.14 (Pin_14); no longer J2.3 (Pin_3)
- net PA3: now also J2.13 (Pin_13); no longer J2.4 (Pin_4)
- net PA4: now also J2.12 (Pin_12); no longer J2.5 (Pin_5)
- net PA5: now also J2.11 (Pin_11); no longer J2.6 (Pin_6)
- net PA6: now also J2.10 (Pin_10); no longer J2.7 (Pin_7)
- net PA7: now also J2.9 (Pin_9); no longer J2.8 (Pin_8)
- net PB10: now also J2.8 (Pin_8); no longer J2.9 (Pin_9)
- net PB5: now also J2.3 (Pin_3); no longer J2.14 (Pin_14)
- net PB6: now also J2.4 (Pin_4); no longer J2.13 (Pin_13)
- net PB7: now also J2.5 (Pin_5); no longer J2.12 (Pin_12)
- net PB8: now also J2.6 (Pin_6); no longer J2.11 (Pin_11)
- net PB9: now also J2.7 (Pin_7); no longer J2.10 (Pin_10)
- net PC0: now also J5.16 (Pin_16); no longer J5.1 (Pin_1)
- net PC1: now also J5.15 (Pin_15); no longer J5.2 (Pin_2)
- net PC2: now also J5.14 (Pin_14); no longer J5.3 (Pin_3)
- net PD5: now also J5.13 (Pin_13); no longer J5.4 (Pin_4)
- net PD6: now also J5.12 (Pin_12); no longer J5.5 (Pin_5)
- net PD7: now also J5.11 (Pin_11); no longer J5.6 (Pin_6)
- net PE0: now also J5.10 (Pin_10); no longer J5.7 (Pin_7)
- net PE1: now also J5.9 (Pin_9); no longer J5.8 (Pin_8)
- net PE2: now also J5.8 (Pin_8); no longer J5.9 (Pin_9)
- net PE3: now also J5.7 (Pin_7); no longer J5.10 (Pin_10)
- net PE6: now also J5.6 (Pin_6); no longer J5.11 (Pin_11)
- net PE7: now also J5.5 (Pin_5); no longer J5.12 (Pin_12)
- net PF0: now also J5.1 (Pin_1); no longer J5.16 (Pin_16)
- net PF1: now also J5.2 (Pin_2); no longer J5.15 (Pin_15)
- net PF2: now also J5.3 (Pin_3); no longer J5.14 (Pin_14)
- net PF3: now also J5.4 (Pin_4); no longer J5.13 (Pin_13)
- net PF4_MODE0: now also J6.3 (Pin_3); no longer J6.9 (Pin_9)
- net PF5_MODE1: now also J6.4 (Pin_4); no longer J6.8 (Pin_8)
- net PF6_MODE2: now also J6.5 (Pin_5); no longer J6.7 (Pin_7)
- net VUSB: now also J6.2 (Pin_2); no longer J3.9 (Pin_9)
- net WAKEUP: now also J3.4 (Pin_4); no longer J6.1 (Pin_1)
- net nRESET: now also J3.5 (Pin_5); no longer J3.6 (Pin_6)

Commit message: update footprints
Parts:
- J1: footprint Connector_PinHeader_2.54mm:PinHeader_1x04_P2.54mm_Vertical -> Connector_PinHeader_2.54mm:PinHeader_1x04_P2.54mm_Horizontal
- SW1, SW3: footprint Button_Switch_SMD:SW_SPST_CK_RS282G05A3 -> Button_Switch_SMD:SW_SPST_B3U-1000P
Changed lines of the file:
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@@
 			)
 		)
-		(property "Footprint" "Button_Switch_SMD:SW_SPST_CK_RS282G05A3"
+		(property "Footprint" "Button_Switch_SMD:SW_SPST_B3U-1000P"
 			(at 199.39 74.93 0)
 			(effects
@@
 			)
 		)
-		(property "Footprint" "Connector_PinHeader_2.54mm:PinHeader_1x04_P2.54mm_Vertical"
+		(property "Footprint" "Connector_PinHeader_2.54mm:PinHeader_1x04_P2.54mm_Horizontal"
 			(at 196.85 34.29 0)
 			(effects
@@
 			)
 		)
-		(property "Footprint" "Button_Switch_SMD:SW_SPST_CK_RS282G05A3"
+		(property "Footprint" "Button_Switch_SMD:SW_SPST_B3U-1000P"
 			(at 60.96 171.45 0)
 			(effects

Commit message: part made
Parts:
- C10, C11, C12, C4, C5, C6, C7, C8, C9: footprint Capacitor_SMD:C_0603_1608Metric -> Capacitor_SMD:C_0402_1005Metric
- D3, D5: footprint LED_SMD:LED_0805_2012Metric -> LED_SMD:LED_0603_1608Metric
- R1, R10, R11, R12, R13, R14, R15, R16, R17, R18, R19, R2, R20, R21, R22, R3, R4, R5, R6, R7, R8, R9: footprint Resistor_SMD:R_0603_1608Metric -> Resistor_SMD:R_0402_1005Metric
Changed lines of the file:
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@@
 			)
 		)
-		(property "Footprint" "LED_SMD:LED_0805_2012Metric"
+		(property "Footprint" "LED_SMD:LED_0603_1608Metric"
 			(at 200.66 106.68 0)
 			(effects
@@
 			)
 		)
-		(property "Footprint" "Capacitor_SMD:C_0603_1608Metric"
+		(property "Footprint" "Capacitor_SMD:C_0402_1005Metric"
 			(at 134.3152 176.53 0)
 			(effects
@@
 			)
 		)
-		(property "Footprint" "Capacitor_SMD:C_0603_1608Metric"
+		(property "Footprint" "Capacitor_SMD:C_0402_1005Metric"
 			(at 103.8352 93.98 0)
 			(effects
@@
 			)
 		)
-		(property "Footprint" "Resistor_SMD:R_0603_1608Metric"
+		(property "Footprint" "Resistor_SMD:R_0402_1005Metric"
 			(at 107.95 80.518 90)
 			(effects
@@
 			)
 		)
-		(property "Footprint" "Resistor_SMD:R_0603_1608Metric"
+		(property "Footprint" "Resistor_SMD:R_0402_1005Metric"
 			(at 210.82 141.478 90)
 			(effects
@@
 			)
 		)
-		(property "Footprint" "Resistor_SMD:R_0603_1608Metric"
+		(property "Footprint" "Resistor_SMD:R_0402_1005Metric"
 			(at 107.95 39.878 90)
 			(effects
@@
 			)
 		)
-		(property "Footprint" "Resistor_SMD:R_0603_1608Metric"
+		(property "Footprint" "Resistor_SMD:R_0402_1005Metric"
 			(at 107.95 50.038 90)
 			(effects
@@
 			)
 		)
-		(property "Footprint" "Resistor_SMD:R_0603_1608Metric"
+		(property "Footprint" "Resistor_SMD:R_0402_1005Metric"
 			(at 109.22 116.078 90)
 			(effects
@@
 			)
 		)
-		(property "Footprint" "Resistor_SMD:R_0603_1608Metric"
+		(property "Footprint" "Resistor_SMD:R_0402_1005Metric"
 			(at 107.95 70.358 90)
 			(effects
@@
 			)
 		)
-		(property "Footprint" "Capacitor_SMD:C_0603_1608Metric"
+		(property "Footprint" "Capacitor_SMD:C_0402_1005Metric"
 			(at 150.8252 86.36 0)
 			(effects
@@
 			)
 		)
-		(property "Footprint" "Resistor_SMD:R_0603_1608Metric"
+		(property "Footprint" "Resistor_SMD:R_0402_1005Metric"
 			(at 107.95 85.598 90)
 			(effects
@@
 			)
 		)
-		(property "Footprint" "Capacitor_SMD:C_0603_1608Metric"
+		(property "Footprint" "Capacitor_SMD:C_0402_1005Metric"
 			(at 110.1852 176.53 0)
 			(effects
@@
 			)
 		)
-		(property "Footprint" "Capacitor_SMD:C_0603_1608Metric"
+		(property "Footprint" "Capacitor_SMD:C_0402_1005Metric"
 			(at 133.0452 43.18 0)
 			(effects
@@
 			)
 		)
-		(property "Footprint" "Resistor_SMD:R_0603_1608Metric"
+		(property "Footprint" "Resistor_SMD:R_0402_1005Metric"
 			(at 107.95 55.118 90)
 			(effects
@@
 			)
 		)
-		(property "Footprint" "Capacitor_SMD:C_0603_1608Metric"
+		(property "Footprint" "Capacitor_SMD:C_0402_1005Metric"
 			(at 122.8852 176.53 0)
 			(effects
@@
 			)
 		)
-		(property "Footprint" "Resistor_SMD:R_0603_1608Metric"
+		(property "Footprint" "Resistor_SMD:R_0402_1005Metric"
 			(at 107.95 75.438 90)
 			(effects
@@
 			)
 		)
-		(property "Footprint" "Resistor_SMD:R_0603_1608Metric"
+		(property "Footprint" "Resistor_SMD:R_0402_1005Metric"
 			(at 109.22 121.158 90)
 			(effects
@@
 			)
 		)
-		(property "Footprint" "Capacitor_SMD:C_0603_1608Metric"
+		(property "Footprint" "Capacitor_SMD:C_0402_1005Metric"
 			(at 153.3652 43.18 0)
 			(effects
@@
 			)
 		)
-		(property "Footprint" "Resistor_SMD:R_0603_1608Metric"
+		(property "Footprint" "Resistor_SMD:R_0402_1005Metric"
 			(at 82.042 172.72 90)
 			(effects
@@
 			)
 		)
-		(property "Footprint" "Resistor_SMD:R_0603_1608Metric"
+		(property "Footprint" "Resistor_SMD:R_0402_1005Metric"
 			(at 68.072 181.61 90)
 			(effects
@@
 			)
 		)
-		(property "Footprint" "Capacitor_SMD:C_0603_1608Metric"
+		(property "Footprint" "Capacitor_SMD:C_0402_1005Metric"
 			(at 167.3352 176.53 0)
 			(effects
@@
 			)
 		)
-		(property "Footprint" "Resistor_SMD:R_0603_1608Metric"
+		(property "Footprint" "Resistor_SMD:R_0402_1005Metric"
 			(at 107.95 29.718 90)
 			(effects
@@
 			)
 		)
-		(property "Footprint" "LED_SMD:LED_0805_2012Metric"
+		(property "Footprint" "LED_SMD:LED_0603_1608Metric"
 			(at 83.82 181.61 0)
 			(effects
@@
 			)
 		)
-		(property "Footprint" "Resistor_SMD:R_0603_1608Metric"
+		(property "Footprint" "Resistor_SMD:R_0402_1005Metric"
 			(at 241.3 112.522 90)
 			(effects
@@
 			)
 		)
-		(property "Footprint" "Resistor_SMD:R_0603_1608Metric"
+		(property "Footprint" "Resistor_SMD:R_0402_1005Metric"
 			(at 191.77 108.458 90)
 			(effects
@@
 			)
 		)
-		(property "Footprint" "Resistor_SMD:R_0603_1608Metric"
+		(property "Footprint" "Resistor_SMD:R_0402_1005Metric"
 			(at 107.95 44.958 90)
 			(effects
@@
 			)
 		)
-		(property "Footprint" "Resistor_SMD:R_0603_1608Metric"
+		(property "Footprint" "Resistor_SMD:R_0402_1005Metric"
 			(at 107.95 34.798 90)
 			(effects
@@
 			)
 		)
-		(property "Footprint" "Resistor_SMD:R_0603_1608Metric"
+		(property "Footprint" "Resistor_SMD:R_0402_1005Metric"
 			(at 107.95 60.198 90)
 			(effects
@@
 			)
 		)
-		(property "Footprint" "Capacitor_SMD:C_0603_1608Metric"
+		(property "Footprint" "Capacitor_SMD:C_0402_1005Metric"
 			(at 135.5852 86.36 0)
 			(effects
@@
 			)
 		)
-		(property "Footprint" "Resistor_SMD:R_0603_1608Metric"
+		(property "Footprint" "Resistor_SMD:R_0402_1005Metric"
 			(at 241.3 118.872 90)
 			(effects
@@
 			)
 		)
-		(property "Footprint" "Resistor_SMD:R_0603_1608Metric"
+		(property "Footprint" "Resistor_SMD:R_0402_1005Metric"
 			(at 107.95 65.278 90)
 			(effects
@@
 			)
 		)
-		(property "Footprint" "Resistor_SMD:R_0603_1608Metric"
+		(property "Footprint" "Resistor_SMD:R_0402_1005Metric"
 			(at 109.22 110.998 90)
 			(effects
@@
 			)
 		)
-		(property "Footprint" "Resistor_SMD:R_0603_1608Metric"
+		(property "Footprint" "Resistor_SMD:R_0402_1005Metric"
 			(at 187.452 73.66 90)
 			(effects

Commit message: exclude battery holder
Parts:
- removed BT1: CR1220, MDR32-K1986BE92FI-DK:MPD_BC501SM-TR, symbol Device:Battery_Cell
- renumbered C12 to C11, C11 to C12
Connections:
- net +BATT_SRC: now also J2.2 (Pin_2); no longer J3.3 (Pin_3)
- net GND: now also J3.3 (Pin_3); no longer J2.2 (Pin_2)
Other:
- moved on the sheet: C11

Commit message: update cap sizes
Parts:
- C10, C11, C12, C4, C5, C6, C7, C8, C9: footprint Capacitor_SMD:C_0402_1005Metric -> Capacitor_SMD:C_0603_1608Metric
Changed lines of the file:
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@@
 			)
 		)
-		(property "Footprint" "Capacitor_SMD:C_0402_1005Metric"
+		(property "Footprint" "Capacitor_SMD:C_0603_1608Metric"
 			(at 134.3152 176.53 0)
 			(effects
@@
 			)
 		)
-		(property "Footprint" "Capacitor_SMD:C_0402_1005Metric"
+		(property "Footprint" "Capacitor_SMD:C_0603_1608Metric"
 			(at 103.8352 93.98 0)
 			(effects
@@
 			)
 		)
-		(property "Footprint" "Capacitor_SMD:C_0402_1005Metric"
+		(property "Footprint" "Capacitor_SMD:C_0603_1608Metric"
 			(at 150.8252 86.36 0)
 			(effects
@@
 			)
 		)
-		(property "Footprint" "Capacitor_SMD:C_0402_1005Metric"
+		(property "Footprint" "Capacitor_SMD:C_0603_1608Metric"
 			(at 110.1852 176.53 0)
 			(effects
@@
 			)
 		)
-		(property "Footprint" "Capacitor_SMD:C_0402_1005Metric"
+		(property "Footprint" "Capacitor_SMD:C_0603_1608Metric"
 			(at 133.0452 43.18 0)
 			(effects
@@
 			)
 		)
-		(property "Footprint" "Capacitor_SMD:C_0402_1005Metric"
+		(property "Footprint" "Capacitor_SMD:C_0603_1608Metric"
 			(at 122.8852 176.53 0)
 			(effects
@@
 			)
 		)
-		(property "Footprint" "Capacitor_SMD:C_0402_1005Metric"
+		(property "Footprint" "Capacitor_SMD:C_0603_1608Metric"
 			(at 153.3652 43.18 0)
 			(effects
@@
 			)
 		)
-		(property "Footprint" "Capacitor_SMD:C_0402_1005Metric"
+		(property "Footprint" "Capacitor_SMD:C_0603_1608Metric"
 			(at 152.0952 176.53 0)
 			(effects
@@
 			)
 		)
-		(property "Footprint" "Capacitor_SMD:C_0402_1005Metric"
+		(property "Footprint" "Capacitor_SMD:C_0603_1608Metric"
 			(at 135.5852 86.36 0)
 			(effects

Commit message: update resistors sizes
Parts:
- R1, R10, R11, R12, R13, R14, R15, R16, R17, R18, R19, R2, R20, R21, R22, R3, R4, R5, R6, R7, R8, R9: footprint Resistor_SMD:R_0402_1005Metric -> Resistor_SMD:R_0603_1608Metric
Changed lines of the file:
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@@
 			)
 		)
-		(property "Footprint" "Resistor_SMD:R_0402_1005Metric"
+		(property "Footprint" "Resistor_SMD:R_0603_1608Metric"
 			(at 107.95 80.518 90)
 			(effects
@@
 			)
 		)
-		(property "Footprint" "Resistor_SMD:R_0402_1005Metric"
+		(property "Footprint" "Resistor_SMD:R_0603_1608Metric"
 			(at 210.82 141.478 90)
 			(effects
@@
 			)
 		)
-		(property "Footprint" "Resistor_SMD:R_0402_1005Metric"
+		(property "Footprint" "Resistor_SMD:R_0603_1608Metric"
 			(at 107.95 39.878 90)
 			(effects
@@
 			)
 		)
-		(property "Footprint" "Resistor_SMD:R_0402_1005Metric"
+		(property "Footprint" "Resistor_SMD:R_0603_1608Metric"
 			(at 107.95 50.038 90)
 			(effects
@@
 			)
 		)
-		(property "Footprint" "Resistor_SMD:R_0402_1005Metric"
+		(property "Footprint" "Resistor_SMD:R_0603_1608Metric"
 			(at 109.22 116.078 90)
 			(effects
@@
 			)
 		)
-		(property "Footprint" "Resistor_SMD:R_0402_1005Metric"
+		(property "Footprint" "Resistor_SMD:R_0603_1608Metric"
 			(at 107.95 70.358 90)
 			(effects
@@
 			)
 		)
-		(property "Footprint" "Resistor_SMD:R_0402_1005Metric"
+		(property "Footprint" "Resistor_SMD:R_0603_1608Metric"
 			(at 107.95 85.598 90)
 			(effects
@@
 			)
 		)
-		(property "Footprint" "Resistor_SMD:R_0402_1005Metric"
+		(property "Footprint" "Resistor_SMD:R_0603_1608Metric"
 			(at 107.95 55.118 90)
 			(effects
@@
 			)
 		)
-		(property "Footprint" "Resistor_SMD:R_0402_1005Metric"
+		(property "Footprint" "Resistor_SMD:R_0603_1608Metric"
 			(at 107.95 75.438 90)
 			(effects
@@
 			)
 		)
-		(property "Footprint" "Resistor_SMD:R_0402_1005Metric"
+		(property "Footprint" "Resistor_SMD:R_0603_1608Metric"
 			(at 109.22 121.158 90)
 			(effects
@@
 			)
 		)
-		(property "Footprint" "Resistor_SMD:R_0402_1005Metric"
+		(property "Footprint" "Resistor_SMD:R_0603_1608Metric"
 			(at 82.042 172.72 90)
 			(effects
@@
 			)
 		)
-		(property "Footprint" "Resistor_SMD:R_0402_1005Metric"
+		(property "Footprint" "Resistor_SMD:R_0603_1608Metric"
 			(at 68.072 181.61 90)
 			(effects
@@
 			)
 		)
-		(property "Footprint" "Resistor_SMD:R_0402_1005Metric"
+		(property "Footprint" "Resistor_SMD:R_0603_1608Metric"
 			(at 107.95 29.718 90)
 			(effects
@@
 			)
 		)
-		(property "Footprint" "Resistor_SMD:R_0402_1005Metric"
+		(property "Footprint" "Resistor_SMD:R_0603_1608Metric"
 			(at 241.3 112.522 90)
 			(effects
@@
 			)
 		)
-		(property "Footprint" "Resistor_SMD:R_0402_1005Metric"
+		(property "Footprint" "Resistor_SMD:R_0603_1608Metric"
 			(at 191.77 108.458 90)
 			(effects
@@
 			)
 		)
-		(property "Footprint" "Resistor_SMD:R_0402_1005Metric"
+		(property "Footprint" "Resistor_SMD:R_0603_1608Metric"
 			(at 107.95 44.958 90)
 			(effects
@@
 			)
 		)
-		(property "Footprint" "Resistor_SMD:R_0402_1005Metric"
+		(property "Footprint" "Resistor_SMD:R_0603_1608Metric"
 			(at 107.95 34.798 90)
 			(effects
@@
 			)
 		)
-		(property "Footprint" "Resistor_SMD:R_0402_1005Metric"
+		(property "Footprint" "Resistor_SMD:R_0603_1608Metric"
 			(at 107.95 60.198 90)
 			(effects
@@
 			)
 		)
-		(property "Footprint" "Resistor_SMD:R_0402_1005Metric"
+		(property "Footprint" "Resistor_SMD:R_0603_1608Metric"
 			(at 241.3 118.872 90)
 			(effects
@@
 			)
 		)
-		(property "Footprint" "Resistor_SMD:R_0402_1005Metric"
+		(property "Footprint" "Resistor_SMD:R_0603_1608Metric"
 			(at 107.95 65.278 90)
 			(effects
@@
 			)
 		)
-		(property "Footprint" "Resistor_SMD:R_0402_1005Metric"
+		(property "Footprint" "Resistor_SMD:R_0603_1608Metric"
 			(at 109.22 110.998 90)
 			(effects
@@
 			)
 		)
-		(property "Footprint" "Resistor_SMD:R_0402_1005Metric"
+		(property "Footprint" "Resistor_SMD:R_0603_1608Metric"
 			(at 187.452 73.66 90)
 			(effects
