File: MDR32-K1986BE92FI-DK/MDR32-K1986BE92FI-DK.kicad_sch (KiCad schematic)
At the start: 56 parts, among them J1 Conn_PROBE, J2 PIN_A, J3 SYS_A, J4 USB_C_Receptacle_USB2.0_16P, J5 PIN_B, J6 SYS_B, Q1 AO3401A, SW1 B3U-1000P, SW2 SW_DIP_x02, SW3 B3U-1000P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

Commit message: PinHeader_1x04
Parts:
- J1: symbol Connector_Generic:Conn_01x04 -> MDR32-K1986BE92FI-DK:Conn_01x04
Changed lines of the file:
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@@
 	)
 	(symbol
-		(lib_id "Connector_Generic:Conn_01x04")
+		(lib_id "MDR32-K1986BE92FI-DK:Conn_01x04")
 		(at 196.85 34.29 0)
 		(unit 1)

Commit message: SW_Push
Parts:
- SW1, SW3: footprint Button_Switch_SMD:SW_SPST_B3U-1000P -> MDR32-K1986BE92FI-DK:SW_SPST_B3U-1000P; symbol Switch:SW_Push -> MDR32-K1986BE92FI-DK:SW_Push
Changed lines of the file:
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@@
 	)
 	(symbol
-		(lib_id "Switch:SW_Push")
+		(lib_id "MDR32-K1986BE92FI-DK:SW_Push")
 		(at 199.39 80.01 0)
 		(unit 1)
@@
 			)
 		)
-		(property "Footprint" "Button_Switch_SMD:SW_SPST_B3U-1000P"
+		(property "Footprint" "MDR32-K1986BE92FI-DK:SW_SPST_B3U-1000P"
 			(at 199.39 74.93 0)
 			(effects
@@
 	)
 	(symbol
-		(lib_id "Switch:SW_Push")
+		(lib_id "MDR32-K1986BE92FI-DK:SW_Push")
 		(at 60.96 176.53 0)
 		(unit 1)
@@
 			)
 		)
-		(property "Footprint" "Button_Switch_SMD:SW_SPST_B3U-1000P"
+		(property "Footprint" "MDR32-K1986BE92FI-DK:SW_SPST_B3U-1000P"
 			(at 60.96 171.45 0)
 			(effects

Commit message: SW_DIP_x02
Parts:
- SW2: footprint Button_Switch_SMD:SW_DIP_SPSTx02_Slide_Omron_A6H-2101_W6.15mm_P1.27mm -> MDR32-K1986BE92FI-DK:SW_DIP_SPSTx02_Slide_Omron_A6H-2101_W6.15mm_P1.27mm; symbol Switch:SW_DIP_x02 -> MDR32-K1986BE92FI-DK:SW_DIP_x02
Changed lines of the file:
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@@
 	)
 	(symbol
-		(lib_id "Switch:SW_DIP_x02")
+		(lib_id "MDR32-K1986BE92FI-DK:SW_DIP_x02")
 		(at 198.12 139.7 0)
 		(unit 1)
@@
 			)
 		)
-		(property "Footprint" "Button_Switch_SMD:SW_DIP_SPSTx02_Slide_Omron_A6H-2101_W6.15mm_P1.27mm"
+		(property "Footprint" "MDR32-K1986BE92FI-DK:SW_DIP_SPSTx02_Slide_Omron_A6H-2101_W6.15mm_P1.27mm"
 			(at 198.12 139.7 0)
 			(effects

Commit message: Resistors
Parts:
- R1, R10, R11, R12, R13, R14, R15, R16, R17, R18, R19, R2, R20, R21, R22, R3, R4, R5, R6, R7, R8, R9: footprint Resistor_SMD:R_0603_1608Metric -> MDR32-K1986BE92FI-DK:R_0603_1608Metric; symbol Device:R -> MDR32-K1986BE92FI-DK:R
Changed lines of the file:
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@@
 	)
 	(symbol
-		(lib_id "Device:R")
+		(lib_id "MDR32-K1986BE92FI-DK:R")
 		(at 107.95 78.74 90)
 		(unit 1)
@@
 			)
 		)
-		(property "Footprint" "Resistor_SMD:R_0603_1608Metric"
+		(property "Footprint" "MDR32-K1986BE92FI-DK:R_0603_1608Metric"
 			(at 107.95 80.518 90)
 			(effects
@@
 	)
 	(symbol
-		(lib_id "Device:R")
+		(lib_id "MDR32-K1986BE92FI-DK:R")
 		(at 210.82 139.7 90)
 		(unit 1)
@@
 			)
 		)
-		(property "Footprint" "Resistor_SMD:R_0603_1608Metric"
+		(property "Footprint" "MDR32-K1986BE92FI-DK:R_0603_1608Metric"
 			(at 210.82 141.478 90)
 			(effects
@@
 	)
 	(symbol
-		(lib_id "Device:R")
+		(lib_id "MDR32-K1986BE92FI-DK:R")
 		(at 107.95 38.1 90)
 		(unit 1)
@@
 			)
 		)
-		(property "Footprint" "Resistor_SMD:R_0603_1608Metric"
+		(property "Footprint" "MDR32-K1986BE92FI-DK:R_0603_1608Metric"
 			(at 107.95 39.878 90)
 			(effects
@@
 	)
 	(symbol
-		(lib_id "Device:R")
+		(lib_id "MDR32-K1986BE92FI-DK:R")
 		(at 107.95 48.26 90)
 		(unit 1)
@@
 			)
 		)
-		(property "Footprint" "Resistor_SMD:R_0603_1608Metric"
+		(property "Footprint" "MDR32-K1986BE92FI-DK:R_0603_1608Metric"
 			(at 107.95 50.038 90)
 			(effects
@@
 	)
 	(symbol
-		(lib_id "Device:R")
+		(lib_id "MDR32-K1986BE92FI-DK:R")
 		(at 109.22 114.3 90)
 		(unit 1)
@@
 			)
 		)
-		(property "Footprint" "Resistor_SMD:R_0603_1608Metric"
+		(property "Footprint" "MDR32-K1986BE92FI-DK:R_0603_1608Metric"
 			(at 109.22 116.078 90)
 			(effects
@@
 	)
 	(symbol
-		(lib_id "Device:R")
+		(lib_id "MDR32-K1986BE92FI-DK:R")
 		(at 107.95 68.58 90)
 		(unit 1)
@@
 			)
 		)
-		(property "Footprint" "Resistor_SMD:R_0603_1608Metric"
+		(property "Footprint" "MDR32-K1986BE92FI-DK:R_0603_1608Metric"
 			(at 107.95 70.358 90)
 			(effects
@@
 	)
 	(symbol
-		(lib_id "Device:R")
+		(lib_id "MDR32-K1986BE92FI-DK:R")
 		(at 107.95 83.82 90)
 		(unit 1)
@@
 			)
 		)
-		(property "Footprint" "Resistor_SMD:R_0603_1608Metric"
+		(property "Footprint" "MDR32-K1986BE92FI-DK:R_0603_1608Metric"
 			(at 107.95 85.598 90)
 			(effects
@@
 	)
 	(symbol
-		(lib_id "Device:R")
+		(lib_id "MDR32-K1986BE92FI-DK:R")
 		(at 107.95 53.34 90)
 		(unit 1)
@@
 			)
 		)
-		(property "Footprint" "Resistor_SMD:R_0603_1608Metric"
+		(property "Footprint" "MDR32-K1986BE92FI-DK:R_0603_1608Metric"
 			(at 107.95 55.118 90)
 			(effects
@@
 	)
 	(symbol
-		(lib_id "Device:R")
+		(lib_id "MDR32-K1986BE92FI-DK:R")
 		(at 107.95 73.66 90)
 		(unit 1)
@@
 			)
 		)
-		(property "Footprint" "Resistor_SMD:R_0603_1608Metric"
+		(property "Footprint" "MDR32-K1986BE92FI-DK:R_0603_1608Metric"
 			(at 107.95 75.438 90)
 			(effects
@@
 	)
 	(symbol
-		(lib_id "Device:R")
+		(lib_id "MDR32-K1986BE92FI-DK:R")
 		(at 109.22 119.38 90)
 		(unit 1)
@@
 			)
 		)
-		(property "Footprint" "Resistor_SMD:R_0603_1608Metric"
+		(property "Footprint" "MDR32-K1986BE92FI-DK:R_0603_1608Metric"
 			(at 109.22 121.158 90)
 			(effects
@@
 	)
 	(symbol
-		(lib_id "Device:R")
+		(lib_id "MDR32-K1986BE92FI-DK:R")
 		(at 83.82 172.72 0)
 		(unit 1)
@@
 			)
 		)
-		(property "Footprint" "Resistor_SMD:R_0603_1608Metric"
+		(property "Footprint" "MDR32-K1986BE92FI-DK:R_0603_1608Metric"
 			(at 82.042 172.72 90)
 			(effects
@@
 	)
 	(symbol
-		(lib_id "Device:R")
+		(lib_id "MDR32-K1986BE92FI-DK:R")
 		(at 69.85 181.61 0)
 		(unit 1)
@@
 			)
 		)
-		(property "Footprint" "Resistor_SMD:R_0603_1608Metric"
+		(property "Footprint" "MDR32-K1986BE92FI-DK:R_0603_1608Metric"
 			(at 68.072 181.61 90)
 			(effects
@@
 	)
 	(symbol
-		(lib_id "Device:R")
+		(lib_id "MDR32-K1986BE92FI-DK:R")
 		(at 107.95 27.94 90)
 		(unit 1)
@@
 			)
 		)
-		(property "Footprint" "Resistor_SMD:R_0603_1608Metric"
+		(property "Footprint" "MDR32-K1986BE92FI-DK:R_0603_1608Metric"
 			(at 107.95 29.718 90)
 			(effects
@@
 	)
 	(symbol
-		(lib_id "Device:R")
+		(lib_id "MDR32-K1986BE92FI-DK:R")
 		(at 241.3 114.3 270)
 		(unit 1)
@@
 			)
 		)
-		(property "Footprint" "Resistor_SMD:R_0603_1608Metric"
+		(property "Footprint" "MDR32-K1986BE92FI-DK:R_0603_1608Metric"
 			(at 241.3 112.522 90)
 			(effects
@@
 	)
 	(symbol
-		(lib_id "Device:R")
+		(lib_id "MDR32-K1986BE92FI-DK:R")
 		(at 191.77 106.68 90)
 		(unit 1)
@@
 			)
 		)
-		(property "Footprint" "Resistor_SMD:R_0603_1608Metric"
+		(property "Footprint" "MDR32-K1986BE92FI-DK:R_0603_1608Metric"
 			(at 191.77 108.458 90)
 			(effects
@@
 	)
 	(symbol
-		(lib_id "Device:R")
+		(lib_id "MDR32-K1986BE92FI-DK:R")
 		(at 107.95 43.18 90)
 		(unit 1)
@@
 			)
 		)
-		(property "Footprint" "Resistor_SMD:R_0603_1608Metric"
+		(property "Footprint" "MDR32-K1986BE92FI-DK:R_0603_1608Metric"
 			(at 107.95 44.958 90)
 			(effects
@@
 	)
 	(symbol
-		(lib_id "Device:R")
+		(lib_id "MDR32-K1986BE92FI-DK:R")
 		(at 107.95 33.02 90)
 		(unit 1)
@@
 			)
 		)
-		(property "Footprint" "Resistor_SMD:R_0603_1608Metric"
+		(property "Footprint" "MDR32-K1986BE92FI-DK:R_0603_1608Metric"
 			(at 107.95 34.798 90)
 			(effects
@@
 	)
 	(symbol
-		(lib_id "Device:R")
+		(lib_id "MDR32-K1986BE92FI-DK:R")
 		(at 107.95 58.42 90)
 		(unit 1)
@@
 			)
 		)
-		(property "Footprint" "Resistor_SMD:R_0603_1608Metric"
+		(property "Footprint" "MDR32-K1986BE92FI-DK:R_0603_1608Metric"
 			(at 107.95 60.198 90)
 			(effects
@@
 	)
 	(symbol
-		(lib_id "Device:R")
+		(lib_id "MDR32-K1986BE92FI-DK:R")
 		(at 241.3 120.65 270)
 		(unit 1)
@@
 			)
 		)
-		(property "Footprint" "Resistor_SMD:R_0603_1608Metric"
+		(property "Footprint" "MDR32-K1986BE92FI-DK:R_0603_1608Metric"
 			(at 241.3 118.872 90)
 			(effects
@@
 	)
 	(symbol
-		(lib_id "Device:R")
+		(lib_id "MDR32-K1986BE92FI-DK:R")
 		(at 107.95 63.5 90)
 		(unit 1)
@@
 			)
 		)
-		(property "Footprint" "Resistor_SMD:R_0603_1608Metric"
+		(property "Footprint" "MDR32-K1986BE92FI-DK:R_0603_1608Metric"
 			(at 107.95 65.278 90)
 			(effects
@@
 	)
 	(symbol
-		(lib_id "Device:R")
+		(lib_id "MDR32-K1986BE92FI-DK:R")
 		(at 109.22 109.22 90)
 		(unit 1)
@@
 			)
 		)
-		(property "Footprint" "Resistor_SMD:R_0603_1608Metric"
+		(property "Footprint" "MDR32-K1986BE92FI-DK:R_0603_1608Metric"
 			(at 109.22 110.998 90)
 			(effects
@@
 	)
 	(symbol
-		(lib_id "Device:R")
+		(lib_id "MDR32-K1986BE92FI-DK:R")
 		(at 189.23 73.66 0)
 		(unit 1)
@@
 			)
 		)
-		(property "Footprint" "Resistor_SMD:R_0603_1608Metric"
+		(property "Footprint" "MDR32-K1986BE92FI-DK:R_0603_1608Metric"
 			(at 187.452 73.66 90)
 			(effects

Commit message: SOT-23
Parts:
- D3: footprint Package_TO_SOT_SMD:SOT-23 -> MDR32-K1986BE92FI-DK:SOT-23; symbol Diode:BAT54C -> MDR32-K1986BE92FI-DK:BAT54C
- Q1: footprint Package_TO_SOT_SMD:SOT-23 -> MDR32-K1986BE92FI-DK:SOT-23; symbol Transistor_FET:AO3401A -> MDR32-K1986BE92FI-DK:AO3401A
Changed lines of the file:
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@@
 	)
 	(symbol
-		(lib_id "Transistor_FET:AO3401A")
+		(lib_id "MDR32-K1986BE92FI-DK:AO3401A")
 		(at 69.85 170.18 270)
 		(mirror x)
@@
 			)
 		)
-		(property "Footprint" "Package_TO_SOT_SMD:SOT-23"
+		(property "Footprint" "MDR32-K1986BE92FI-DK:SOT-23"
 			(at 67.945 165.1 0)
 			(effects
@@
 	)
 	(symbol
-		(lib_id "Diode:BAT54C")
+		(lib_id "MDR32-K1986BE92FI-DK:BAT54C")
 		(at 180.34 137.16 0)
 		(mirror x)
@@
 			)
 		)
-		(property "Footprint" "Package_TO_SOT_SMD:SOT-23"
+		(property "Footprint" "MDR32-K1986BE92FI-DK:SOT-23"
 			(at 182.245 140.335 0)
 			(effects

Commit message: SolderJumper
Parts:
- JP1, JP2: footprint Jumper:SolderJumper-2_P1.3mm_Open_TrianglePad1.0x1.5mm -> MDR32-K1986BE92FI-DK:SolderJumper-2_P1.3mm_Open_TrianglePad1.0x1.5mm; symbol Jumper:SolderJumper_2_Open -> MDR32-K1986BE92FI-DK:SolderJumper_2_Open
Changed lines of the file:
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@@
 	)
 	(symbol
-		(lib_id "Jumper:SolderJumper_2_Open")
+		(lib_id "MDR32-K1986BE92FI-DK:SolderJumper_2_Open")
 		(at 144.78 118.11 0)
 		(unit 1)
@@
 			)
 		)
-		(property "Footprint" "Jumper:SolderJumper-2_P1.3mm_Open_TrianglePad1.0x1.5mm"
+		(property "Footprint" "MDR32-K1986BE92FI-DK:SolderJumper-2_P1.3mm_Open_TrianglePad1.0x1.5mm"
 			(at 144.78 118.11 0)
 			(effects
@@
 	)
 	(symbol
-		(lib_id "Jumper:SolderJumper_2_Open")
+		(lib_id "MDR32-K1986BE92FI-DK:SolderJumper_2_Open")
 		(at 144.78 109.22 0)
 		(unit 1)
@@
 			)
 		)
-		(property "Footprint" "Jumper:SolderJumper-2_P1.3mm_Open_TrianglePad1.0x1.5mm"
-			(at 144.78 110.49 0)
-			(effects
-				(font
+		(property "Footprint" "MDR32-K1986BE92FI-DK:SolderJumper-2_P1.3mm_Open_TrianglePad1.0x1.5mm"
+			(at 144.78 109.22 0)
+			(effects
+				(font

Commit message: PinHeader
Parts:
- J2, J5: footprint Connector_PinHeader_2.54mm:PinHeader_1x16_P2.54mm_Vertical -> MDR32-K1986BE92FI-DK:PinHeader_1x16_P2.54mm_Vertical; symbol Connector_Generic:Conn_01x16 -> MDR32-K1986BE92FI-DK:Conn_01x16
- J3, J6: footprint Connector_PinHeader_2.54mm:PinHeader_1x10_P2.54mm_Vertical -> MDR32-K1986BE92FI-DK:PinHeader_1x10_P2.54mm_Vertical; symbol Connector_Generic:Conn_01x10 -> MDR32-K1986BE92FI-DK:Conn_01x10
Changed lines of the file:
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@@
 	)
 	(symbol
-		(lib_id "Connector_Generic:Conn_01x10")
+		(lib_id "MDR32-K1986BE92FI-DK:Conn_01x10")
 		(at 242.57 80.01 0)
 		(mirror x)
@@
 			)
 		)
-		(property "Footprint" "Connector_PinHeader_2.54mm:PinHeader_1x10_P2.54mm_Vertical"
+		(property "Footprint" "MDR32-K1986BE92FI-DK:PinHeader_1x10_P2.54mm_Vertical"
 			(at 242.57 80.01 0)
 			(effects
@@
 	)
 	(symbol
-		(lib_id "Connector_Generic:Conn_01x10")
+		(lib_id "MDR32-K1986BE92FI-DK:Conn_01x10")
 		(at 271.78 80.01 0)
 		(mirror x)
@@
 			)
 		)
-		(property "Footprint" "Connector_PinHeader_2.54mm:PinHeader_1x10_P2.54mm_Vertical"
+		(property "Footprint" "MDR32-K1986BE92FI-DK:PinHeader_1x10_P2.54mm_Vertical"
 			(at 271.78 80.01 0)
 			(effects
@@
 	)
 	(symbol
-		(lib_id "Connector_Generic:Conn_01x16")
+		(lib_id "MDR32-K1986BE92FI-DK:Conn_01x16")
 		(at 271.78 43.18 0)
 		(mirror x)
@@
 			)
 		)
-		(property "Footprint" "Connector_PinHeader_2.54mm:PinHeader_1x16_P2.54mm_Vertical"
+		(property "Footprint" "MDR32-K1986BE92FI-DK:PinHeader_1x16_P2.54mm_Vertical"
 			(at 271.78 43.18 0)
 			(effects
@@
 	)
 	(symbol
-		(lib_id "Connector_Generic:Conn_01x16")
+		(lib_id "MDR32-K1986BE92FI-DK:Conn_01x16")
 		(at 242.57 43.18 0)
 		(mirror x)
@@
 			)
 		)
-		(property "Footprint" "Connector_PinHeader_2.54mm:PinHeader_1x16_P2.54mm_Vertical"
+		(property "Footprint" "MDR32-K1986BE92FI-DK:PinHeader_1x16_P2.54mm_Vertical"
 			(at 242.57 43.18 0)
 			(effects

Commit message: Fuse
Parts:
- F1, F2: footprint Fuse:Fuse_0603_1608Metric -> MDR32-K1986BE92FI-DK:Fuse_0603_1608Metric; symbol Device:Polyfuse -> MDR32-K1986BE92FI-DK:Polyfuse
Changed lines of the file:
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@@
 	)
 	(symbol
-		(lib_id "Device:Polyfuse")
+		(lib_id "MDR32-K1986BE92FI-DK:Polyfuse")
 		(at 240.03 151.13 0)
 		(unit 1)
@@
 			)
 		)
-		(property "Footprint" "Fuse:Fuse_0603_1608Metric"
+		(property "Footprint" "MDR32-K1986BE92FI-DK:Fuse_0603_1608Metric"
 			(at 241.3 156.21 0)
 			(effects
@@
 	)
 	(symbol
-		(lib_id "Device:Polyfuse")
+		(lib_id "MDR32-K1986BE92FI-DK:Polyfuse")
 		(at 246.38 151.13 0)
 		(unit 1)
@@
 			)
 		)
-		(property "Footprint" "Fuse:Fuse_0603_1608Metric"
+		(property "Footprint" "MDR32-K1986BE92FI-DK:Fuse_0603_1608Metric"
 			(at 247.65 156.21 0)
 			(effects
