File: MDR32-K1986BE92FI-DK/MDR32-K1986BE92FI-DK.kicad_sch (KiCad schematic)
At the start: 56 parts, among them J1 Conn_PROBE, J2 PIN_A, J3 SYS_A, J4 USB_C_Receptacle_USB2.0_16P, J5 PIN_B, J6 SYS_B, Q1 AO3401A, SW1 IT-1181, SW2 SW_DIP_x02, SW3 IT-1181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

Commit message: update LED sizes
Parts:
- D3, D5: footprint LED_SMD:LED_0603_1608Metric -> LED_SMD:LED_0805_2012Metric
Changed lines of the file:
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@@
 			)
 		)
-		(property "Footprint" "LED_SMD:LED_0603_1608Metric"
+		(property "Footprint" "LED_SMD:LED_0805_2012Metric"
 			(at 200.66 106.68 0)
 			(effects
@@
 			)
 		)
-		(property "Footprint" "LED_SMD:LED_0603_1608Metric"
+		(property "Footprint" "LED_SMD:LED_0805_2012Metric"
 			(at 83.82 181.61 0)
 			(effects

Commit message: part position
Connections:
- net WAKEUP: now also J3.5 (Pin_5); no longer J3.4 (Pin_4)
- net nRESET: now also J3.4 (Pin_4); no longer J3.5 (Pin_5)
Changed lines of the file:
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@@
 	)
 	(label "nRESET"
-		(at 229.87 80.01 0)
+		(at 229.87 82.55 0)
 		(fields_autoplaced yes)
 		(effects
@@
 	)
 	(label "WAKEUP"
-		(at 229.87 82.55 0)
+		(at 229.87 80.01 0)
 		(fields_autoplaced yes)
 		(effects

Commit message: part route
Connections:
- net JATDI: now also J3.9 (Pin_9); no longer J3.7 (Pin_7)
- net JATDO: now also J3.6 (Pin_6); no longer J3.10 (Pin_10)
- net JATMS: now also J3.7 (Pin_7); no longer J3.9 (Pin_9)
- net JAnTRS: now also J3.10 (Pin_10); no longer J3.6 (Pin_6)
- net PC0: now also J5.1 (Pin_1); no longer J5.16 (Pin_16)
- net PC1: now also J5.2 (Pin_2); no longer J5.15 (Pin_15)
- net PC2: now also J5.3 (Pin_3); no longer J5.14 (Pin_14)
- net PD5: now also J5.4 (Pin_4); no longer J5.13 (Pin_13)
- net PD6: now also J5.5 (Pin_5); no longer J5.12 (Pin_12)
- net PD7: now also J5.6 (Pin_6); no longer J5.11 (Pin_11)
- net PE0: now also J5.7 (Pin_7); no longer J5.10 (Pin_10)
- net PE1: now also J5.8 (Pin_8); no longer J5.9 (Pin_9)
- net PE2: now also J5.9 (Pin_9); no longer J5.8 (Pin_8)
- net PE3: now also J5.10 (Pin_10); no longer J5.7 (Pin_7)
- net PE6: now also J5.11 (Pin_11); no longer J5.6 (Pin_6)
- net PE7: now also J5.12 (Pin_12); no longer J5.5 (Pin_5)
- net PF0: now also J5.16 (Pin_16); no longer J5.1 (Pin_1)
- net PF1: now also J5.15 (Pin_15); no longer J5.2 (Pin_2)
- net PF2: now also J5.14 (Pin_14); no longer J5.3 (Pin_3)
- net PF3: now also J5.13 (Pin_13); no longer J5.4 (Pin_4)
Changed lines of the file:
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@@
 	)
 	(label "PC0"
-		(at 259.08 22.86 0)
+		(at 259.08 60.96 0)
 		(fields_autoplaced yes)
 		(effects
@@
 	)
 	(label "PF3"
-		(at 259.08 53.34 0)
+		(at 259.08 30.48 0)
 		(fields_autoplaced yes)
 		(effects
@@
 	)
 	(label "PC1"
-		(at 259.08 25.4 0)
+		(at 259.08 58.42 0)
 		(fields_autoplaced yes)
 		(effects
@@
 	)
 	(label "JAnTRS"
-		(at 229.87 77.47 0)
+		(at 229.87 67.31 0)
 		(fields_autoplaced yes)
 		(effects
@@
 	)
 	(label "PE6"
-		(at 259.08 48.26 0)
+		(at 259.08 35.56 0)
 		(fields_autoplaced yes)
 		(effects
@@
 	)
 	(label "PD7"
-		(at 259.08 35.56 0)
+		(at 259.08 48.26 0)
 		(fields_autoplaced yes)
 		(effects
@@
 	)
 	(label "JATDO"
-		(at 229.87 67.31 0)
+		(at 229.87 77.47 0)
 		(fields_autoplaced yes)
 		(effects
@@
 	)
 	(label "PF0"
-		(at 259.08 60.96 0)
+		(at 259.08 22.86 0)
 		(fields_autoplaced yes)
 		(effects
@@
 	)
 	(label "PC2"
-		(at 259.08 27.94 0)
+		(at 259.08 55.88 0)
 		(fields_autoplaced yes)
 		(effects
@@
 	)
 	(label "PE2"
-		(at 259.08 43.18 0)
+		(at 259.08 40.64 0)
 		(fields_autoplaced yes)
 		(effects
@@
 	)
 	(label "PE3"
-		(at 259.08 45.72 0)
+		(at 259.08 38.1 0)
 		(fields_autoplaced yes)
 		(effects
@@
 	)
 	(label "PE7"
+		(at 259.08 33.02 0)
+		(fields_autoplaced yes)
+		(effects
+			(font
+				(size 1.27 1.27)
+			)
+			(justify left bottom)
+		)
+	)
+	(label "PD6"
 		(at 259.08 50.8 0)
-		(fields_autoplaced yes)
-		(effects
-			(font
-				(size 1.27 1.27)
-			)
-			(justify left bottom)
-		)
-	)
-	(label "PD6"
-		(at 259.08 33.02 0)
 		(fields_autoplaced yes)
 		(effects
@@
 	)
 	(label "JATDI"
-		(at 229.87 74.93 0)
+		(at 229.87 69.85 0)
 		(fields_autoplaced yes)
 		(effects
@@
 	)
 	(label "PF1"
-		(at 259.08 58.42 0)
+		(at 259.08 25.4 0)
 		(fields_autoplaced yes)
 		(effects
@@
 	)
 	(label "PF2"
-		(at 259.08 55.88 0)
+		(at 259.08 27.94 0)
 		(fields_autoplaced yes)
 		(effects
@@
 	)
 	(label "PD5"
-		(at 259.08 30.48 0)
+		(at 259.08 53.34 0)
 		(fields_autoplaced yes)
 		(effects
@@
 	)
 	(label "PE1"
-		(at 259.08 40.64 0)
+		(at 259.08 43.18 0)
 		(fields_autoplaced yes)
 		(effects
@@
 	)
 	(label "JATMS"
-		(at 229.87 69.85 0)
+		(at 229.87 74.93 0)
 		(fields_autoplaced yes)
 		(effects
@@
 	)
 	(label "PE0"
-		(at 259.08 38.1 0)
-		(fields_autoplaced yes)
-		(effects
+		(at 259.08 45.72 0)
+		(fields_autoplaced yes)
+		(effects

Commit message: unctional route and dependencies
Parts:
- removed D2: K1986BE92FI, Package_DFN_QFN:QFN-64-1EP_9x9mm_P0.5mm_EP7.5x7.5mm, symbol MDR32-K1986BE92FI-DK:K1986BE92FI
- removed U1: LM1117GS-3.3, Package_TO_SOT_SMD:SOT-223-3_TabPin2, symbol Regulator_Linear:AMS1117-3.3
- added U1: LM1117GS-3.3, Package_TO_SOT_SMD:SOT-223, symbol MDR32-K1986BE92FI-DK:LM1117MP-3.3
- added U2: K1986BE92FI, Package_DFN_QFN:QFN-64-1EP_9x9mm_P0.5mm_EP7.5x7.5mm, symbol MDR32-K1986BE92FI-DK:K1986BE92FI
- J1: footprint Connector_PinHeader_2.54mm:PinHeader_1x04_P2.54mm_Horizontal -> MDR32-K1986BE92FI-DK:PinHeader_1x04_P2.54mm_Horizontal
- J4: footprint Connector_USB:USB_C_Receptacle_GCT_USB4105-xx-A_16P_TopMnt_Horizontal -> MDR32-K1986BE92FI-DK:USB_C_Receptacle_GCT_USB4105-xx-A_16P_TopMnt_Horizontal
- renumbered D3 to D2, D4 to D3, D5 to D4
Connections:
- net +3V3: now also U2.1 (+3V3), U2.24 (AUCC1), U2.28 (AUCC)
- net +BATT: now also U2.13 (BUCC)
- net GND: now also U1.1 (GND), U2.11 (GND), U2.23 (AGND1), U2.27 (AGND), U2.39 (GND), U2.49 (GND), U2.64 (GND), U2.65 (PAD)
- net JATCK: now also U2.45 (PB2)
- net JATDI: now also U2.46 (PB3)
- net JATDO: now also U2.43 (PB0)
- net JATMS: now also U2.44 (PB1)
- net JAnTRS: now also U2.47 (PB4)
- net JBTCK: now also U2.32 (PD1)
- net JBTDI: now also U2.34 (PD3)
- net JBTDO: now also U2.30 (PD4)
- net JBTMS: now also U2.31 (PD0)
- net JBnTRS: now also U2.33 (PD2)
- net OSC_IN: now also U2.19 (OSC_IN)
- net OSC_IN32: now also U2.16 (PE6)
- net OSC_OUT: now also U2.20 (OSC_OUT)
- net OSC_OUT32: now also U2.15 (PE7)
- net PA0: now also U2.63 (PA0)
- net PA1: now also U2.62 (PA1)
- net PA2: now also U2.61 (PA2)
- net PA3: now also U2.60 (PA3)
- net PA4: now also U2.59 (PA4)
- net PA5: now also U2.58 (PA5)
- net PA6: now also U2.57 (PA6)
- net PA7: now also U2.56 (PA7)
- net PB10: now also U2.55 (PB10)
- net PB5: now also U2.50 (PB5)
- net PB6: now also U2.51 (PB6)
- net PB7: now also U2.52 (PB7)
- net PB8: now also U2.53 (PB8)
- net PB9: now also U2.54 (PB9)
- net PC0: now also U2.42 (PC0)
- net PC1: now also U2.41 (PC1)
- net PC2: now also U2.40 (PC2)
- net PD5: now also U2.35 (PD5)
- net PD6: now also U2.36 (PD6)
- net PD7: now also U2.29 (PD7)
- net PE0: now also U2.26 (PE0)
- net PE1: now also U2.25 (PE1)
- net PE2: now also U2.22 (PE2)
- net PE3: now also U2.21 (PE3)
- net PF0: now also U2.2 (PF0)
- net PF1: now also U2.3 (PF1)
- net PF2: now also U2.4 (PF2)
- net PF3: now also U2.5 (PF3)
- net PF4_MODE0: now also U2.6 (PF4)
- net PF5_MODE1: now also U2.7 (PF5)
- net PF6_MODE2: now also U2.8 (PF6)
- net USBDN: now also U2.10 (DN)
- net USBDP: now also U2.9 (DP)
- net VUSB: now also U1.3 (VI)
- net WAKEUP: now also U2.17 (WAKEUP)
- net nRESET: now also U2.18 (~{RESET})
- net at D1.2 (A): now also U1.2 (VO)

Commit message: update net list
Parts:
- C12, C7: value 12pF -> 10pF
- SW1, SW3: value IT-1181 -> B3U-1000P
Changed lines of the file:
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@@
 			)
 		)
-		(property "Value" "IT-1181"
+		(property "Value" "B3U-1000P"
 			(at 199.39 85.598 0)
 			(effects
@@
 			)
 		)
-		(property "Value" "12pF"
+		(property "Value" "10pF"
 			(at 135.89 40.6399 0)
 			(effects
@@
 			)
 		)
-		(property "Value" "12pF"
+		(property "Value" "10pF"
 			(at 156.21 40.6399 0)
 			(effects
@@
 			)
 		)
-		(property "Value" "IT-1181"
+		(property "Value" "B3U-1000P"
 			(at 60.96 171.45 0)
 			(effects

Commit message: fix 3d model for QFN-64
Parts:
- U2: footprint Package_DFN_QFN:QFN-64-1EP_9x9mm_P0.5mm_EP7.5x7.5mm -> MDR32-K1986BE92FI-DK:QFN-64-1EP_9x9mm_P0.5mm_EP7.5x7.5mm
Changed lines of the file:
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@@
 			)
 		)
-		(property "Footprint" "Package_DFN_QFN:QFN-64-1EP_9x9mm_P0.5mm_EP7.5x7.5mm"
+		(property "Footprint" "MDR32-K1986BE92FI-DK:QFN-64-1EP_9x9mm_P0.5mm_EP7.5x7.5mm"
 			(at 50.8 145.034 0)
 			(effects

Commit message: Move local for archive (#1)
Move symbol and footprint to local for archive
Parts:
- C1, C2: footprint Capacitor_SMD:C_0805_2012Metric -> MDR32-K1986BE92FI-DK:C_0805_2012Metric; symbol Device:C -> MDR32-K1986BE92FI-DK:C
- C10, C11, C12, C4, C5, C6, C7, C8, C9: footprint Capacitor_SMD:C_0603_1608Metric -> MDR32-K1986BE92FI-DK:C_0603_1608Metric; symbol Device:C -> MDR32-K1986BE92FI-DK:C
- C3: footprint Capacitor_Tantalum_SMD:CP_EIA-3216-18_Kemet-A -> MDR32-K1986BE92FI-DK:CP_EIA-3216-18_Kemet-A; symbol Device:C_Polarized -> MDR32-K1986BE92FI-DK:C_Polarized
- D1: footprint Diode_SMD:D_SOD-123 -> MDR32-K1986BE92FI-DK:D_SOD-123; symbol Device:D_Filled -> MDR32-K1986BE92FI-DK:D_Filled
- D2, D4: footprint LED_SMD:LED_0805_2012Metric -> MDR32-K1986BE92FI-DK:LED_0805_2012Metric; symbol Device:LED -> MDR32-K1986BE92FI-DK:LED
- D3: footprint Package_TO_SOT_SMD:SOT-23 -> MDR32-K1986BE92FI-DK:SOT-23; symbol Diode:BAT54C -> MDR32-K1986BE92FI-DK:BAT54C
- F1, F2: footprint Fuse:Fuse_0603_1608Metric -> MDR32-K1986BE92FI-DK:Fuse_0603_1608Metric; symbol Device:Polyfuse -> MDR32-K1986BE92FI-DK:Polyfuse
- J1: symbol Connector_Generic:Conn_01x04 -> MDR32-K1986BE92FI-DK:Conn_01x04
- J2, J5: footprint Connector_PinHeader_2.54mm:PinHeader_1x16_P2.54mm_Vertical -> MDR32-K1986BE92FI-DK:PinHeader_1x16_P2.54mm_Vertical; symbol Connector_Generic:Conn_01x16 -> MDR32-K1986BE92FI-DK:Conn_01x16
- J3, J6: footprint Connector_PinHeader_2.54mm:PinHeader_1x10_P2.54mm_Vertical -> MDR32-K1986BE92FI-DK:PinHeader_1x10_P2.54mm_Vertical; symbol Connector_Generic:Conn_01x10 -> MDR32-K1986BE92FI-DK:Conn_01x10
- J4: symbol Connector:USB_C_Receptacle_USB2.0_16P -> MDR32-K1986BE92FI-DK:USB_C_Receptacle_USB2.0_16P
- JP1, JP2: footprint Jumper:SolderJumper-2_P1.3mm_Open_TrianglePad1.0x1.5mm -> MDR32-K1986BE92FI-DK:SolderJumper-2_P1.3mm_Open_TrianglePad1.0x1.5mm; symbol Jumper:SolderJumper_2_Open -> MDR32-K1986BE92FI-DK:SolderJumper_2_Open
- Q1: footprint Package_TO_SOT_SMD:SOT-23 -> MDR32-K1986BE92FI-DK:SOT-23; symbol Transistor_FET:AO3401A -> MDR32-K1986BE92FI-DK:AO3401A
- R1, R10, R11, R12, R13, R14, R15, R16, R17, R18, R19, R2, R20, R21, R22, R3, R4, R5, R6, R7, R8, R9: footprint Resistor_SMD:R_0603_1608Metric -> MDR32-K1986BE92FI-DK:R_0603_1608Metric; symbol Device:R -> MDR32-K1986BE92FI-DK:R
- SW1, SW3: footprint Button_Switch_SMD:SW_SPST_B3U-1000P -> MDR32-K1986BE92FI-DK:SW_SPST_B3U-1000P; symbol Switch:SW_Push -> MDR32-K1986BE92FI-DK:SW_Push
- SW2: footprint Button_Switch_SMD:SW_DIP_SPSTx02_Slide_Omron_A6H-2101_W6.15mm_P1.27mm -> MDR32-K1986BE92FI-DK:SW_DIP_SPSTx02_Slide_Omron_A6H-2101_W6.15mm_P1.27mm; symbol Switch:SW_DIP_x02 -> MDR32-K1986BE92FI-DK:SW_DIP_x02
- U1: footprint Package_TO_SOT_SMD:SOT-223 -> MDR32-K1986BE92FI-DK:SOT-223; symbol MDR32-K1986BE92FI-DK:LM1117MP-3.3 -> MDR32-K1986BE92FI-DK:LM1117GS-3.3
- Y1: footprint Crystal:Crystal_SMD_3225-4Pin_3.2x2.5mm -> MDR32-K1986BE92FI-DK:Crystal_SMD_3225-4Pin_3.2x2.5mm; symbol Device:Crystal_GND24 -> MDR32-K1986BE92FI-DK:Crystal_GND24
- Y2: footprint Crystal:Crystal_SMD_3215-2Pin_3.2x1.5mm -> MDR32-K1986BE92FI-DK:Crystal_SMD_3215-2Pin_3.2x1.5mm; symbol Device:Crystal -> MDR32-K1986BE92FI-DK:Crystal

Commit message: rename
Parts:
- C3: value 22µF -> T491A226K006AT 22µF
- D2: value LED -> GREEN
- D4: value LED -> BLUE
- J4: value USB_C_Receptacle_USB2.0_16P -> USB4105-GF-A USB2.0 16P
- SW2: value SW_DIP_x02 -> DHN-02-T-V
- Y1: value SMD3225 P4 16MHz -> X322516MLB4SI SMD3225 P4 16MHz
- Y2: value 32.768KHz ±20ppm 6pF -> NX3215SA 32.768KHz ±20ppm 6pF
Changed lines of the file:
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@@
 			)
 		)
-		(property "Value" "LED"
+		(property "Value" "BLUE"
 			(at 198.755 109.855 0)
 			(effects
@@
 			)
 		)
-		(property "Value" "USB_C_Receptacle_USB2.0_16P"
+		(property "Value" "USB4105-GF-A USB2.0 16P"
 			(at 267.97 109.22 0)
 			(effects
@@
 			)
 		)
-		(property "Value" "SMD3225 P4  16MHz"
+		(property "Value" "X322516MLB4SI SMD3225 P4  16MHz"
 			(at 142.24 22.86 0)
 			(effects
@@
 			)
 		)
-		(property "Value" "SW_DIP_x02"
+		(property "Value" "DHN-02-T-V"
 			(at 198.12 132.08 0)
 			(effects
@@
 		(on_board yes)
 		(dnp no)
-		(fields_autoplaced yes)
 		(property "Reference" "C3"
 			(at 100.33 170.5609 0)
@@
 			)
 		)
-		(property "Value" "22µF"
-			(at 100.33 173.1009 0)
+		(property "Value" "T491A226K006AT 22µF"
+			(at 86.36 176.53 0)
 			(effects
 				(font
@@
 			)
 		)
-		(property "Value" "LED"
+		(property "Value" "GREEN"
 			(at 87.63 184.4674 90)
 			(effects
@@
 			)
 		)
-		(property "Value" "32.768KHz ±20ppm 6pF"
+		(property "Value" "NX3215SA 32.768KHz ±20ppm 6pF"
 			(at 142.24 68.58 0)
 			(effects
