File: MDR32-K1986BE92FI-DK/MDR32-K1986BE92FI-DK.kicad_pcb (KiCad board)
At the start: 2 copper layers, 69.6 x 21.4 mm, 56 parts, among them J1 Conn_PROBE, J2 PIN_A, J3 SYS_A, J4 USB_C_Receptacle_USB2.0_16P, J5 PIN_B, J6 SYS_B, Q1 AO3401A, SW1 IT-1181, SW2 SW_DIP_x02, SW3 IT-1181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

Commit message: part position
Parts:
- C1, C2, D1, D4, U1: moved to F.Cu
- moved R17 30.7 mm to (30.8, 22.3), turned to -90 degrees
- moved R16 29.8 mm to (29.4, 22.3), turned to -90 degrees
- moved R15 28.9 mm to (27.9, 22.3), turned to -90 degrees
- moved R12 27.2 mm to (32.3, 22.3), turned to -90 degrees
- moved U1 27.0 mm to (36.4, 27.7)
- moved R11 25.3 mm to (33.8, 22.3), turned to -90 degrees
- moved C1 24.6 mm to (31.0, 29.0), turned to 90 degrees
- moved C4 23.8 mm to (27.9, 33.2), turned to 90 degrees
- moved R10 23.5 mm to (35.2, 22.3), turned to -90 degrees
- moved C2 22.1 mm to (28.2, 29.0), turned to -90 degrees
- moved R14 21.8 mm to (29.4, 33.2), turned to 90 degrees
- moved R9 21.6 mm to (36.7, 22.3), turned to -90 degrees
- moved R8 19.8 mm to (38.1, 22.3), turned to -90 degrees
- moved D1 19.8 mm to (29.6, 26.1)
- moved R13 19.7 mm to (30.8, 33.2), turned to 90 degrees
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Connections:
- J3 pad 4: /WAKEUP -> /nRESET
- J3 pad 5: /nRESET -> /WAKEUP

Commit message: part position
Parts:
- moved C8 23.8 mm to (50.4, 47.5)
- moved C11 23.8 mm to (50.4, 49.1)
- moved C6 22.3 mm to (50.4, 46.1)
- moved C5 20.8 mm to (50.4, 44.6)
- moved C3 19.1 mm to (50.3, 42.8)
- moved R1 11.6 mm to (41.1, 33.2), turned to -90 degrees
- moved D4 11.0 mm to (44.2, 22.0)
- moved C2 11.0 mm to (39.3, 29.4), turned to 90 degrees
- moved R2 9.44 mm to (39.6, 33.2), turned to -90 degrees
- moved C1 8.78 mm to (39.3, 26.0), turned to -90 degrees
- moved R19 7.95 mm to (41.1, 22.3), turned to -90 degrees
- moved D1 7.68 mm to (37.1, 27.7), turned to 90 degrees
- moved D5 7.53 mm to (41.2, 26.0), turned to 90 degrees
- moved D3 7.38 mm to (41.2, 29.4), turned to -90 degrees
- moved U1 4.81 mm to (31.6, 27.7), turned to 180 degrees
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
Commit message: part position
Parts:
- moved C8 29.9 mm to (68.6, 23.8), turned to 45 degrees
- moved C6 29.2 mm to (66.9, 21.9), turned to 45 degrees
- moved C11 25.7 mm to (69.1, 31.4), turned to -45 degrees
- moved C5 17.4 mm to (54.8, 27.7), turned to -90 degrees
- moved C3 15.3 mm to (53.0, 27.7), turned to -90 degrees
- moved R18 3.04 mm to (48.1, 24.5), turned to 0 degrees
- moved SW3 1.17 mm to (48.0, 22.1)
- moved SW1 1.16 mm to (48.0, 33.3)
- moved D4 0.49 mm to (43.7, 22.1)
- moved Q1 0.38 mm to (43.7, 33.4)

Commit message: part position
Parts:
- JP1, JP2: moved to B.Cu
- moved Y2 24.5 mm to (73.8, 28.6)
- moved JP1 23.0 mm to (73.3, 28.5), turned to 180 degrees
- moved JP2 23.0 mm to (73.3, 32.0), turned to 180 degrees
- moved C10 20.1 mm to (72.4, 30.4), turned to 0 degrees
- moved C9 19.9 mm to (75.5, 30.5), turned to 180 degrees
- moved C12 19.7 mm to (76.5, 25.7)
- moved C7 19.7 mm to (70.8, 25.7)
- moved Y1 19.7 mm to (73.6, 25.7)
- moved C6 0.48 mm to (66.4, 21.9)
- moved C11 0.43 mm to (69.2, 30.9)
- turned R2 to 90 degrees

Commit message: start route
Routing:
- net +3V3: track 0.00 -> 18.9 mm
- net VUSB: track 0.00 -> 15.8 mm
- net GND: track 0.00 -> 10.9 mm
- net Net-(D1-A): track 0.00 -> 10.0 mm
- net Net-(D3-A): track 0.00 -> 3.11 mm
- net +3V3_SRC: track 0.00 -> 3.00 mm
- net /USBDP: track 2.81 -> 4.90 mm
- net /USBDN: track 3.08 -> 5.17 mm
- net Net-(D5-A): track 0.00 -> 2.00 mm
- net /nRESET: track 0.00 -> 1.48 mm

Commit message: part route
Parts:
- moved R11 4.38 mm to (38.1, 22.3)
- moved R8 4.38 mm to (33.8, 22.3)
- turned R21 to 90 degrees
- turned R22 to -90 degrees
Routing:
- net +3V3_SRC: track 3.00 -> 32.5 mm, vias 0 -> 1
- net /PA0: track 0.00 -> 25.6 mm
- net /PA1: track 0.00 -> 23.8 mm
- net /PA2: track 0.00 -> 22.7 mm
- net /PA3: track 0.00 -> 20.9 mm
- net VUSB: track 15.8 -> 31.7 mm, vias 0 -> 3
- net /PB8: track 0.00 -> 13.1 mm
- net /PB7: track 0.00 -> 13.1 mm
- net /PB6: track 0.00 -> 10.4 mm
- net /PB5: track 0.00 -> 10.4 mm
- net Net-(Q1-G): track 0.00 -> 6.97 mm
- net /PB9: track 0.00 -> 6.60 mm
- net /PB10: track 0.00 -> 5.69 mm
- net /PF4_MODE0: track 0.00 -> 5.30 mm
- net Net-(J4-CC1): track 0.00 -> 5.18 mm
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
Commit message: part route
Parts:
- moved C10 17.9 mm to (72.4, 12.6)
- moved C11 17.9 mm to (69.2, 13.1)
- moved C12 17.9 mm to (76.4, 7.83)
- moved C3 17.9 mm to (53.0, 9.88)
- moved C5 17.9 mm to (54.8, 9.88)
- moved C9 17.9 mm to (75.4, 12.6)
- moved JP1 17.9 mm to (73.3, 10.6)
- moved JP2 17.9 mm to (73.3, 14.2)
- moved Y1 17.9 mm to (73.6, 7.83)
- moved Y2 17.9 mm to (73.8, 10.7)
- moved C7 17.9 mm to (70.7, 7.82)
- moved C8 11.7 mm to (57.0, 22.1), turned to 135 degrees
- moved C6 11.6 mm to (55.1, 24.3), turned to 135 degrees
- moved R6 5.84 mm to (32.3, 33.2)
- moved R7 5.84 mm to (38.1, 33.2)
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Connections:
- J3 pad 10: /JATDO -> /JAnTRS
- J3 pad 6: /JAnTRS -> /JATDO
- J3 pad 7: /JATDI -> /JATMS
- J3 pad 9: /JATMS -> /JATDI
- J5 pad 1: /PF0 -> /PC0
- J5 pad 10: /PE0 -> /PE3
- J5 pad 11: /PD7 -> /PE6
- J5 pad 12: /PD6 -> /PE7
- J5 pad 13: /PD5 -> /PF3
- J5 pad 14: /PC2 -> /PF2
- J5 pad 15: /PC1 -> /PF1
- J5 pad 16: /PC0 -> /PF0
- J5 pad 2: /PF1 -> /PC1
- J5 pad 3: /PF2 -> /PC2
- J5 pad 4: /PF3 -> /PD5
- J5 pad 5: /PE7 -> /PD6
- J5 pad 6: /PE6 -> /PD7
- J5 pad 7: /PE3 -> /PE0
- J5 pad 8: /PE2 -> /PE1
- J5 pad 9: /PE1 -> /PE2
Routing:
- net /PA5: track 0.00 -> 10.1 mm
- net /PA4: track 2.47 -> 12.6 mm, vias 1 -> 0
- net /PA6: track 0.00 -> 7.74 mm
- net /PA7: track 0.00 -> 6.48 mm
- net /PA3: track 20.9 -> 15.0 mm
- net /PA2: track 22.7 -> 17.4 mm
- net /PB8: track 13.1 -> 8.61 mm
- net /PA1: track 23.8 -> 19.8 mm
- net /PA0: track 25.6 -> 22.2 mm
- net /PB5: track 10.4 -> 13.6 mm
- net /PB7: track 13.1 -> 10.3 mm
- net /JAnTRS: track 2.95 -> 5.02 mm
- net /JATDO: track 5.02 -> 2.95 mm
- net /PB6: track 10.4 -> 12.0 mm
- net /JATMS: track 3.93 -> 2.77 mm
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
Commit message: part route
Parts:
- moved C3 26.1 mm to (71.8, 27.9)
- moved C5 23.6 mm to (70.0, 27.9)
- moved C6 0.90 mm to (55.9, 23.9)
- moved C8 0.49 mm to (57.2, 22.6)
Routing:
- net /JATMS: track 2.77 -> 57.2 mm, vias 0 -> 1
- net /JATCK: track 3.21 -> 52.9 mm, vias 0 -> 1
- net /JATDO: track 2.95 -> 33.2 mm, vias 0 -> 1
- net /JATDI: track 3.93 -> 27.2 mm, vias 0 -> 1
- net /JAnTRS: track 5.02 -> 26.0 mm, vias 0 -> 1
- net /PC2: track 0.00 -> 11.9 mm
- net /PD5: track 0.00 -> 9.79 mm
- net VUSB: track 31.7 -> 33.5 mm
