File: MDR32-K1986BE92FI-KeyBrain-v0.2/MDR32-K1986BE92FI-KeyBrain.kicad_pcb (KiCad board)
At the start: 4 copper layers, 18.1 x 33.3 mm, 40 parts, among them J1 USB-C USB 2.0 MC-372, J2 SWD, U1 AP2112K-3.3, U2 USBLC6-2SC6, U3 K1986BE92FI, U4 ProMicro, Y1 8MHz

Commit message: Исправил подписи пинов
Parts:
- moved REF** 1.00 mm to (80.8, 71.0)
Routing:
- net GND: vias 17 -> 19
Other:
- board text added: "3v3"
- board text added: "CLK"
- board text added: "DIO"
- board text added: "GND"
- board text added: "JTAG 1"
- board text added: "JTAG 2"
- board text added: "JTAG 3"
